File: 0006_Relay_Module_ALDP105.kicad_sch (KiCad schematic)
At the start: 32 parts, among them J1 Screw_Terminal_01x02, K1 ALDP105W, K2 ALDP105W, K3 ALDP105W, K4 ALDP105W, Q1 BC817, U1 TLP185

Commit message: Add files via upload
Parts:
- removed D2: LED, LED_SMD:LED_0805_2012Metric, symbol Device:LED
- removed D8: 1N5819W, 1n5819W:SODFL3618X110N, symbol 1N5819W:1N5819W
- removed J1: Screw_Terminal_01x02, TerminalBlock_Phoenix:TerminalBlock_Phoenix_MKDS-1,5-2-5.08_1x02_P5.08mm_Horizontal, symbol Connector:Screw_Terminal_01x02
- removed K4: ALDP105W, aldp105w:RELAY_ALDP105W, symbol ALDP105W:ALDP105W
- removed Q1: BC817, Package_TO_SOT_SMD:SOT-23, symbol Transistor_BJT:BC817
- removed R1: 1k, Resistor_SMD:R_0805_2012Metric, symbol Device:R
- removed R2: 220r, Resistor_SMD:R_0805_2012Metric, symbol Device:R
- removed U1: TLP185, Package_SO:SOIC-4_4.55x3.7mm_P2.54mm, symbol Isolator:TLP185
- added D9: LED, LED_SMD:LED_0805_2012Metric, symbol Device:LED
- added R9: R, Resistor_SMD:R_0805_2012Metric, symbol Device:R
- added U5: ~, Moduler_:pin_header_5-3, symbol moduler_pin:air
- J1: footprint TerminalBlock_Phoenix:TerminalBlock_Phoenix_MKDS-1,5-2-5.08_1x02_P5.08mm_Horizontal -> TerminalBlock_4Ucon:TerminalBlock_4Ucon_1x02_P3.50mm_Horizontal
Connections:
- net +5V: now also R9.1, U5.7
- net GND: now also D9.1 (K), U5.9
- net R1: now also U5.12
- net R2: now also U5.13
- net R3: now also U5.14
- net R4: now also U5.15
- new net: D9.2 (A), R9.2
- no-connect marks 0 -> 12
Other:
- note added: "AIR PIN"
- note added: "RELAY"
- moved on the sheet: D2, D4, D7, J1, K1, K2, K3, Q1, R1, R2, U1
